File: suruq-keyboard-pcb.kicad_pcb (KiCad board)
At the start: 2 copper layers, 304.8 x 100.7 mm, 150 parts, among them J1 AVR-ISP-6, SW1 Esc, SW10 9, SW11 0, SW12 -, SW13 =, SW14 Back, SW15 Tab, SW16 Q, SW17 W, SW18 E, SW19 R, SW2 1, SW20 T, SW21 Y, SW22 U, SW23 I, SW24 O, SW25 P, SW26 [ {, SW27 ] }, SW28 Enter, SW29 Caps Lock, SW3 2, SW30 A, SW31 S, SW32 D, SW33 F, SW34 G, SW35 H, SW36 J, SW37 K, SW38 L, SW39 ; :, SW4 3, SW40 ' @, SW41 ] }, SW42 Up, SW43 L Shifth, SW44 \ |, SW45 Z, SW46 X, SW47 C, SW48 V, SW49 B, SW5 4, SW50 N, SW51 M, SW52 , <, SW53 . >, SW54 / ?, SW55 R Shift, SW56 Down, SW57 L Ctrl, SW58 Home, SW59 L Alt, SW6 5, SW60 Space, SW61 R Alt, SW62 Fn, SW63 Left, SW64 Right, SW65 SW_Push, SW66 Rotary, SW7 6, SW8 7, SW9 8, U1 PRTR5V0U2X, U2 ATmega32U4-AU, Y1 16MHz

Commit message: routing gauche et MCU
Parts:
- moved D8 6.01 mm to (204.3, 106.8)
- moved J1 3.82 mm to (178.2, 177.4)
- moved R6 3.19 mm to (217.5, 183.7)
- moved C5 2.72 mm to (241.1, 174.7)
- moved C4 2.72 mm to (241.1, 177.6)
- moved SW65 2.32 mm to (165.6, 176.1)
- moved R5 2.00 mm to (169.9, 181.1)
- moved C7 1.91 mm to (224.5, 165.9)
- moved F1 1.81 mm to (210.1, 109.4), turned to 90 degrees
- moved Y1 1.43 mm to (236.7, 176.2), turned to 90 degrees
- moved C3 0.68 mm to (235.6, 171.1), turned to 270 degrees
- moved R2 0.59 mm to (210.3, 99.5)
- moved C2 0.55 mm to (213.9, 179.6), turned to 90 degrees
Connections:
- U2 pad 1: row0 -> row3
- U2 pad 36: col6 -> col5
- U2 pad 37: col5 -> col6
- U2 pad 38: row1 -> row4
- U2 pad 39: row4 -> row0
- U2 pad 40: row3 -> row1
Routing:
- net row2: track 0.00 -> 476.3 mm, vias 0 -> 2
- net row4: track 0.00 -> 474.7 mm, vias 0 -> 2
- net row3: track 0.00 -> 409.7 mm, vias 0 -> 2
- net row0: track 272.9 -> 492.6 mm
- net GND: track 0.00 -> 201.5 mm, vias 0 -> 8
- net row1: track 279.4 -> 480.1 mm
- net col0: track 81.1 -> 249.7 mm, vias 0 -> 1
- net +5V: track 0.00 -> 159.2 mm, vias 0 -> 6
- net col1: track 87.0 -> 230.2 mm, vias 0 -> 1
- net col2: track 89.0 -> 207.2 mm, vias 0 -> 1
- net col3: track 67.0 -> 181.5 mm, vias 0 -> 1
- net col4: track 67.0 -> 161.5 mm, vias 0 -> 1
- net col5: track 67.0 -> 131.6 mm, vias 0 -> 1
- net col6: track 87.0 -> 116.1 mm, vias 0 -> 1
- net col13: track 80.1 -> 108.0 mm
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- added copper zone on B.Cu, net GND
- added copper zone on F.Cu, net GND
Other:
- board size 304.8 x 100.7 mm -> 304.8 x 101.2 mm
