File: suruq-keyboard-pcb.kicad_pcb (KiCad board)
At the start: 2 copper layers, 304.8 x 101.2 mm, 150 parts, among them J1 AVR-ISP-6, SW1 Esc, SW10 9, SW11 0, SW12 -, SW13 =, SW14 Back, SW15 Tab, SW16 Q, SW17 W, SW18 E, SW19 R, SW2 1, SW20 T, SW21 Y, SW22 U, SW23 I, SW24 O, SW25 P, SW26 [ {, SW27 ] }, SW28 Enter, SW29 Caps Lock, SW3 2, SW30 A, SW31 S, SW32 D, SW33 F, SW34 G, SW35 H, SW36 J, SW37 K, SW38 L, SW39 ; :, SW4 3, SW40 ' @, SW41 ] }, SW42 Up, SW43 L Shifth, SW44 \ |, SW45 Z, SW46 X, SW47 C, SW48 V, SW49 B, SW5 4, SW50 N, SW51 M, SW52 , <, SW53 . >, SW54 / ?, SW55 R Shift, SW56 Down, SW57 L Ctrl, SW58 Home, SW59 L Alt, SW6 5, SW60 Space, SW61 R Alt, SW62 Fn, SW63 Left, SW64 Right, SW65 SW_Push, SW66 Rotary, SW7 6, SW8 7, SW9 8, U1 PRTR5V0U2X, U2 ATmega32U4-AU, Y1 16MHz

Commit message: backup au cas ou
Parts:
- added G***: LOGO, cc:cc, B.Cu at (180.3, 177.9)
Routing:
- net col8: track 126.3 -> 128.0 mm
- net col9: track 112.8 -> 114.5 mm

Commit message: add silk screen, Fader65
Parts:
- added logo: G***, local:logo, F.Cu at (60.1, 94.0)
- added logo_small: G***, local:logo_small, B.Cu at (183.1, 171.1)
- SW1, SW10, SW11, SW12, SW13, SW16, SW17, SW18, SW19, SW2, SW20, SW21, SW22, SW23, SW24, SW25, SW26, SW27, SW3, SW30, SW31, SW32, SW33, SW34, SW35, SW36, SW37, SW38, SW39, SW4, SW40, SW41, SW42, SW44, SW45, SW46, SW47, SW48, SW49, SW5, SW50, SW51, SW52, SW53, SW54, SW56, SW6, SW63, SW64, SW7, SW8, SW9: footprint Button_Switch_Keyboard:SW_Cherry_MX_1.00u_PCB -> mx_suruq:SW_Cherry_MX_1.00u_PCB_NameSilk
- SW14: footprint Button_Switch_Keyboard:SW_Cherry_MX_2.00u_PCB -> mx_suruq:SW_Cherry_MX_2.00u_PCB_NameSilk
- SW15, SW61, SW62: footprint Button_Switch_Keyboard:SW_Cherry_MX_1.50u_PCB -> mx_suruq:SW_Cherry_MX_1.50u_PCB_NameSilk
- SW28: footprint Button_Switch_Keyboard:SW_Cherry_MX_ISOEnter_PCB -> mx_suruq:SW_Cherry_MX_ISOEnter_PCB_NameSilk
- SW29, SW55: footprint Button_Switch_Keyboard:SW_Cherry_MX_1.75u_PCB -> mx_suruq:SW_Cherry_MX_1.75u_PCB_NameSilk
- SW43, SW57, SW58, SW59: footprint Button_Switch_Keyboard:SW_Cherry_MX_1.25u_PCB -> mx_suruq:SW_Cherry_MX_1.25u_PCB_NameSilk
- SW60: footprint Button_Switch_Keyboard:SW_Cherry_MX_6.25u_PCB -> mx_suruq:SW_Cherry_MX_6.25u_PCB_NameSilk
- moved G*** 1.65 mm to (181.9, 178.3)
